Commit message: added IMU
Signed-off-by: TiNredmc <thipok17@gmail.com>

File: description/robot_core.xacro (robot description, xacro)
@@ -20,3 +20,17 @@
 		</visual>
 	</link>
+	<joint name="imu_joint" type="fixed">
+        	<origin xyz="0 0 0" rpy="0 0 0" />
+        	<parent link="base_link" />
+        	<child link="imu_link" />
+    	</joint>
+	<link name="imu_link">
+		<visual>
+      			<origin rpy="0 0 1.5708" xyz="0 0 0"/>
+      			<geometry>
+        			<box size ="0.03 0.03 0.03"/>
+				</geometry>
+      			<material name="white"/>
+    	</visual>
+    </link>
 </robot>

Commit message: removed IMU from URDF (temp)
Signed-off-by: TiNredmc <thipok17@gmail.com>

File: description/robot_core.xacro (robot description, xacro)
@@ -20,17 +20,3 @@
 		</visual>
 	</link>
-	<joint name="imu_joint" type="fixed">
-        	<origin xyz="0 0 0" rpy="0 0 0" />
-        	<parent link="base_link" />
-        	<child link="imu_link" />
-    	</joint>
-	<link name="imu_link">
-		<visual>
-      			<origin rpy="0 0 1.5708" xyz="0 0 0"/>
-      			<geometry>
-        			<box size ="0.03 0.03 0.03"/>
-				</geometry>
-      			<material name="white"/>
-    	</visual>
-    </link>
 </robot>
