Commit message: corrected path to the STL model
Signed-off-by: TiNredmc <thipok17@gmail.com>

File: description/asus_xtion.xacro (robot description, xacro)
@@ -18,5 +18,5 @@
       <origin xyz=" 0 0 0 " rpy="0 0 0" />
       <geometry>
-        <mesh filename="package://test_pkg/meshes/PS1080-E3IWBD001305.stl" scale="0.001 0.001 0.001"/>
+        <mesh filename="package://tlhx_bot/meshes/PS1080-E3IWBD001305.stl" scale="0.001 0.001 0.001"/>
       </geometry>
     </visual>

Commit message: updated robot model
Signed-off-by: TiNredmc <thipok17@gmail.com>

File: description/asus_xtion.xacro (robot description, xacro)
@@ -28,21 +28,7 @@
     </collision>
   </link>
-  <joint name="camera_depth_joint" type="fixed">
-    <origin xyz="-0.04 0 0" rpy="1.5708 -1.5708 0" />
+  <joint name="camera_depth_optical_joint" type="fixed">
+    <origin xyz="-0.04 0 0" rpy="3.1415 3.1415 3.1415" />
     <parent link="camera_link" />
-    <child link="camera_depth_frame" />
-  </joint>
-  <link name="camera_depth_frame">
-    <inertial>
-      <mass value="0.01" />
-      <origin xyz="0 0 0" />
-      <inertia ixx="0.001" ixy="0.0" ixz="0.0"
-        iyy="0.001" iyz="0.0"
-        izz="0.001" />
-    </inertial>
-  </link>
-  <joint name="camera_depth_optical_joint" type="fixed">
-    <origin xyz="0 0 0" rpy="1.5708 3.1415 1.5708" />
-    <parent link="camera_depth_frame" />
     <child link="openni_depth_optical_frame" />
   </joint>

Commit message: updated according to the current robot model
Signed-off-by: TiNredmc <thipok17@gmail.com>

File: description/asus_xtion.xacro (robot description, xacro)
@@ -42,3 +42,17 @@
     </inertial>
   </link>
+ <joint name="laser_joint" type="fixed">
+    <origin xyz="-0.04 0 0" rpy="1.5708 -1.5708 0.0" />
+    <parent link="camera_link" />
+    <child link="laser_frame" />
+  </joint>
+  <link name="laser_frame">
+    <inertial>
+      <mass value="0.001" />
+      <origin xyz="0 0 0" />
+      <inertia ixx="0.0001" ixy="0.0" ixz="0.0"
+        iyy="0.0001" iyz="0.0"
+        izz="0.0001" />
+    </inertial>
+  </link>
 </robot>

Commit message: update for ABU
Signed-off-by: TiNredmc <thipok17@gmail.com>

File: description/asus_xtion.xacro (robot description, xacro)
@@ -43,6 +43,6 @@
   </link>
  <joint name="laser_joint" type="fixed">
-    <origin xyz="-0.04 0 0" rpy="1.5708 -1.5708 0.0" />
-    <parent link="camera_link" />
+    <origin xyz="-0.25 0.0 0" rpy="0.0 -3.1415 0.0" />
+    <parent link="chassis" />
     <child link="laser_frame" />
   </joint>
@@ -50,5 +50,5 @@
     <inertial>
       <mass value="0.001" />
-      <origin xyz="0 0 0" />
+      <origin xyz="0 -0.2 0" />
       <inertia ixx="0.0001" ixy="0.0" ixz="0.0"
         iyy="0.0001" iyz="0.0"

File: description/robot.urdf.xacro (robot description, xacro)
@@ -2,4 +2,4 @@
 <robot xmlns:xacro="http://www.ros.org/wiki/xacro"  name="robot">
     <xacro:include filename="robot_core.xacro" />
-	<xacro:include filename="asus_xtion.xacro" />
+    <xacro:include filename="asus_xtion.xacro" />
 </robot>

File: description/robot_core.xacro (robot description, xacro)
@@ -15,5 +15,5 @@
 			<origin xyz="0 0 0.075"/>
 			<geometry>
-				<box size="0.3 0.2 0.15"/>
+				<box size="0.54 0.54 0.12"/>
 			</geometry>
 			<material name="white"/>
